File: project/НИРС.sch (KiCad schematic (older format))
At the start: 39 parts, among them J10 J10, J7 J7, J8 J8, J9 J9, j6 J6

Commit message: Added files via upload
Parts:
- removed R? (x8): R, symbol R
- removed R? (x6): 100, symbol R
- removed RWA?: BA56-12SRWA, symbol BA56-12SRWA
- removed U? (x2): 74HC595, symbol 74HC595
- added R? (x7): 100, symbol R
- added R? (x7): 4,7K, symbol R
Connections:
- net labels removed: Dig1, Dig2, Dig3, J6_1, J6_2, J7_10, J7_11, J7_13, QA, QB, QC, QD, QE, QF, QG, QH
- wire segments 97 -> 144
- no-connect marks 7 -> 1
Other:
- note added: "Led-матрица 8х8"
- note added: "eeprom"
- note added: "ИК-Дальномер"
- note added: "УЗ-Дальномер"
- moved on the sheet: C?, G1, IC?, J10A, J7, J8, J9, R?, UD1, j6

Commit message: Added files via upload
Parts:
- removed LED?: GNM-7881AUE, symbol GNM-7881AUE
- removed Q? (x8): irlml6401, TO_SOT_Packages_SMD:SOT-23, symbol irlml6401
- removed R? (x8): 100, symbol R
- added JP?: JUMPER3, symbol JUMPER3
- added S? (x4): CONN_servo, symbol CONN_servo
- added SW?: SW_PUSH, symbol SW_PUSH
- R?: value 100 -> 4,7K
Connections:
- net labels added: Echo, J8_A2, PWM1, PWM2, PWM3, PWM4, PWR, Trig, Vin
- net labels removed: GNM_10, GNM_11, GNM_13, GNM_15, GNM_16, GNM_3, GNM_4, GNM_6, J10_0, J10_1, J8_A0, ROW1, ROW2, ROW3, ROW4, ROW5, ROW6, ROW7, ROW8
- wire segments 144 -> 97
Other:
- note removed: "Led-матрица 8х8"
- moved on the sheet: C?, G1, IC?, J10A, J7, J8, J9, R?, UD1, j6

Commit message: Added files via upload
Parts:
- removed SW?: SW_PUSH, symbol SW_PUSH
- added FLASH?: W25Q32BV, WIFIRE:SOIC-8(.208mil), symbol W25Q32BV
- added SW?: SW_PUSH, symbol SW_PUSH
Connections:
- net Echo: now also J10.9 (4); no longer J10.15 (7)
- net GND: now also FLASH?.4 (GND), SW?.2
- net Trig: now also J7.8 (37); no longer J10.5 (2)
- net at J9.3 (P32_RST): now also SW?.1
- net +3V3: now reaches J9.4 (VCC3V3)
- net +3V3: now also FLASH?.3 (/WP), FLASH?.7 (/HOLD), FLASH?.8 (VCC)
- net PIN_35: now reaches J7.4 (35)
- net PIN_35: now also FLASH?.2 (DO)
- net PIN_36: now reaches J7.6 (36)
- net PIN_36: now also FLASH?.5 (DI)
- net PWM2 renamed PIN_5
- net PIN_5: now also FLASH?.6 (CLK)
- new net PIN_7: FLASH?.1 (/CS), J10.15 (7)
- no-connect marks 1 -> 0
Other:
- note added: "SPI_FLASH"
- moved on the sheet: J7
Changed lines of the file:
@@
 L J9 J9
 U 1 1 56DE101C
-P 9675 1150
-F 0 "J9" H 10055 1125 60  0000 C CNN
-F 1 "J9" H 10050 165 60  0000 C CNN
-F 2 "" H 9675 1150 60  0000 C CNN
-F 3 "" H 9675 1150 60  0000 C CNN
-	1    9675 1150
+P 9680 1150
+F 0 "J9" H 10060 1125 60  0000 C CNN
+F 1 "J9" H 10055 165 60  0000 C CNN
+F 2 "" H 9680 1150 60  0000 C CNN
+F 3 "" H 9680 1150 60  0000 C CNN
+	1    9680 1150
 	-1   0    0    -1
 $EndComp
@@
 F 3 "" H 9775 1995 50  0000 C CNN
 	1    9775 1995
-	1    0    0    -1
-$EndComp
-$Comp
-L +5V #PWR04
-U 1 1 56DE3C38
-P 9775 1680
-F 0 "#PWR04" H 9775 1530 50  0001 C CNN
-F 1 "+5V" H 9775 1820 50  0000 C CNN
-F 2 "" H 9775 1680 50  0000 C CNN
-F 3 "" H 9775 1680 50  0000 C CNN
-	1    9775 1680
 	1    0    0    -1
 $EndComp
@@
 Text Label 8795 4810 2    60   ~ 0
 Echo
-Text Label 6790 5870 0    60   ~ 0
+Text Label 6790 5270 0    60   ~ 0
 Echo
 Text Label 8795 4710 2    60   ~ 0
 Trig
-Text Label 6790 4870 0    60   ~ 0
+Text Label 3685 1940 0    60   ~ 0
 Trig
 Text Label 1125 5820 0    60   ~ 0
@@
 L J7 J7
 U 1 1 56DE1469
-P 3985 1300
-F 0 "J7" H 4205 1230 60  0000 C CNN
-F 1 "J7" H 4215 -545 60  0000 C CNN
-F 2 "" H 3985 1300 60  0000 C CNN
-F 3 "" H 3985 1300 60  0000 C CNN
-	1    3985 1300
+P 3980 1040
+F 0 "J7" H 4200 970 60  0000 C CNN
+F 1 "J7" H 4210 -805 60  0000 C CNN
+F 2 "" H 3980 1040 60  0000 C CNN
+F 3 "" H 3980 1040 60  0000 C CNN
+	1    3980 1040
 	1    0    0    -1
 $EndComp
@@
 Text Notes 8805 4430 2    60   ~ 0
 УЗ-Дальномер
-NoConn ~ 9570 1600
 $Comp
 L J10 J10
@@
 $EndComp
 $Sheet
-S 2525 1790 740  760
+S 2520 1530 740  760
 U 56F4BED4
 F0 "7-SEGM" 60
 F1 "file56F4BED3.sch" 60
-F2 "RCLK" I R 3265 1900 60
-F3 "SER" I R 3265 2100 60
-F4 "SRCLK" I R 3265 2500 60
+F2 "RCLK" I R 3260 1640 60
+F3 "SER" I R 3260 1840 60
+F4 "SRCLK" I R 3260 2240 60
 $EndSheet
 $Sheet
@@
 Text Label 6790 5070 0    60   ~ 0
 PWM1
-Text Label 6790 5470 0    60   ~ 0
+Text Label 6545 5470 0    60   ~ 0
 PWM2
 Text Label 6790 5670 0    60   ~ 0
 PWM3
-Text Label 3665 1700 0    60   ~ 0
+Text Label 3660 1440 0    60   ~ 0
 PWM4
 Text Label 5420 1545 0    60   ~ 0
@@
 COL1
 $Comp
-L SW_PUSH SW?
-U 1 1 57109297
-P 10295 1500
-F 0 "SW?" H 10445 1610 50  0000 C CNN
-F 1 "SW_PUSH" H 10295 1420 50  0000 C CNN
-F 2 "" H 10295 1500 50  0000 C CNN
-F 3 "" H 10295 1500 50  0000 C CNN
-	1    10295 1500
-	1    0    0    -1
-$EndComp
-$Comp
-L GND #PWR?
-U 1 1 5710AD20
-P 10705 1530
-F 0 "#PWR?" H 10705 1280 50  0001 C CNN
-F 1 "GND" H 10705 1380 50  0000 C CNN
-F 2 "" H 10705 1530 50  0000 C CNN
-F 3 "" H 10705 1530 50  0000 C CNN
-	1    10705 1530
-	1    0    0    -1
-$EndComp
+L W25Q32BV FLASH?
+U 1 1 5709C5FC
+P 3180 3430
+F 0 "FLASH?" H 3205 2930 60  0000 C CNN
+F 1 "W25Q32BV" H 3180 3480 60  0000 C CNN
+F 2 "WIFIRE:SOIC-8(.208mil)" H 3180 2930 60  0001 C CNN
+F 3 "" H 3180 2930 60  0000 C CNN
+	1    3180 3430
+	1    0    0    -1
+$EndComp
+$Comp
+L +5V #PWR?
+U 1 1 570A1610
+P 10100 1575
+F 0 "#PWR?" H 10100 1425 50  0001 C CNN
+F 1 "+5V" H 10100 1715 50  0000 C CNN
+F 2 "" H 10100 1575 50  0000 C CNN
+F 3 "" H 10100 1575 50  0000 C CNN
+	1    10100 1575
+	1    0    0    -1
+$EndComp
+$Comp
+L +3V3 #PWR?
+U 1 1 570A1B04
+P 9900 1575
+F 0 "#PWR?" H 9900 1425 50  0001 C CNN
+F 1 "+3V3" H 9900 1715 50  0000 C CNN
+F 2 "" H 9900 1575 50  0000 C CNN
+F 3 "" H 9900 1575 50  0000 C CNN
+	1    9900 1575
+	1    0    0    -1
+$EndComp
+$Comp
+L +3V3 #PWR?
+U 1 1 570A25DB
+P 3155 3255
+F 0 "#PWR?" H 3155 3105 50  0001 C CNN
+F 1 "+3V3" H 3155 3395 50  0000 C CNN
+F 2 "" H 3155 3255 50  0000 C CNN
+F 3 "" H 3155 3255 50  0000 C CNN
+	1    3155 3255
+	1    0    0    -1
+$EndComp
+Text Label 2405 3605 0    60   ~ 0
+PIN_35
+Text Label 3980 3805 2    60   ~ 0
+PIN_36
+Text Label 3980 3705 2    60   ~ 0
+PIN_5
+$Comp
+L GND #PWR?
+U 1 1 570ADA6C
+P 2655 3830
+F 0 "#PWR?" H 2655 3580 50  0001 C CNN
+F 1 "GND" H 2655 3680 50  0000 C CNN
+F 2 "" H 2655 3830 50  0000 C CNN
+F 3 "" H 2655 3830 50  0000 C CNN
+	1    2655 3830
+	1    0    0    -1
+$EndComp
+Text Label 2405 3505 0    60   ~ 0
+PIN_7
 Wire Notes Line
 	1700 5240 840  5240
@@
 	9500 3250 9555 3250
 Wire Wire Line
-	9775 1680 9775 1700
-Wire Wire Line
 	7040 5870 6790 5870
 Wire Wire Line
@@
 	4665 5770 7040 5770
 Wire Wire Line
-	9775 1700 9570 1700
-Wire Wire Line
-	9570 1800 9775 1800
-Wire Wire Line
-	3265 2500 3940 2500
-Wire Wire Line
-	3265 2100 3940 2100
-Wire Wire Line
-	3265 1900 3940 1900
-Wire Wire Line
-	3940 1700 3665 1700
-Wire Wire Line
-	3940 1500 3665 1500
+	9575 1800 9775 1800
+Wire Wire Line
+	3260 2240 3935 2240
+Wire Wire Line
+	3260 1840 3935 1840
+Wire Wire Line
+	3260 1640 3935 1640
+Wire Wire Line
+	3935 1440 3660 1440
+Wire Wire Line
+	3935 1240 3660 1240
 Wire Wire Line
 	5325 5370 7040 5370
@@
 	1370 5820 1125 5820
 Wire Wire Line
-	9570 1900 9590 1900
+	9575 1900 9590 1900
 Wire Wire Line
 	9590 1900 9590 1800
 Connection ~ 9590 1800
 Wire Wire Line
-	7040 4870 6790 4870
+	3935 1940 3685 1940
 Connection ~ 10355 3400
 Wire Notes Line
@@
 	7070 1930 7220 1930
 Wire Wire Line
-	9570 2000 9695 2000
+	9575 2000 9695 2000
 Wire Wire Line
 	6820 2030 6820 2085
@@
 	7040 5070 6790 5070
 Wire Wire Line
-	7040 5470 6790 5470
+	7040 5470 6545 5470
 Wire Wire Line
 	7040 5670 6790 5670
@@
 	4330 5970 7040 5970
 Wire Wire Line
-	9570 1500 9995 1500
-Wire Wire Line
-	10595 1500 10705 1500
-Wire Wire Line
-	10705 1500 10705 1530
+	7040 5270 6790 5270
+Wire Wire Line
+	9575 1600 9900 1600
+Wire Wire Line
+	3630 3505 3705 3505
+Wire Wire Line
+	3705 3305 3705 3605
+Wire Wire Line
+	2405 3605 2730 3605
+Wire Wire Line
+	3630 3805 3980 3805
+Wire Wire Line
+	3980 3705 3630 3705
+Wire Wire Line
+	3705 3605 3630 3605
+Connection ~ 3705 3505
+Wire Wire Line
+	2730 3705 2330 3705
+Wire Wire Line
+	2330 3705 2330 3305
+Wire Wire Line
+	2330 3305 3705 3305
+Wire Wire Line
+	3155 3305 3155 3255
+Connection ~ 3155 3305
+Wire Wire Line
+	2730 3805 2655 3805
+Wire Wire Line
+	2655 3805 2655 3830
+Wire Wire Line
+	2730 3505 2405 3505
+Wire Wire Line
+	9575 1500 9675 1500
+Wire Wire Line
+	9675 1500 9675 1250
+Wire Wire Line
+	9675 1250 9800 1250
+$Comp
+L SW_PUSH SW?
+U 1 1 570B0411
+P 10100 1250
+F 0 "SW?" H 10250 1360 50  0000 C CNN
+F 1 "SW_PUSH" H 10100 1170 50  0000 C CNN
+F 2 "" H 10100 1250 50  0000 C CNN
+F 3 "" H 10100 1250 50  0000 C CNN
+	1    10100 1250
+	1    0    0    -1
+$EndComp
+$Comp
+L GND #PWR?
+U 1 1 570B1244
+P 10525 1300
+F 0 "#PWR?" H 10525 1050 50  0001 C CNN
+F 1 "GND" H 10525 1150 50  0000 C CNN
+F 2 "" H 10525 1300 50  0000 C CNN
+F 3 "" H 10525 1300 50  0000 C CNN
+	1    10525 1300
+	1    0    0    -1
+$EndComp
+Wire Wire Line
+	10400 1250 10525 1250
+Wire Wire Line
+	10525 1250 10525 1300
+Wire Wire Line
+	9900 1600 9900 1575
+Wire Wire Line
+	10100 1575 10100 1700
+Wire Wire Line
+	10100 1700 9575 1700
+Text Label 6790 5870 0    60   ~ 0
+PIN_7
+Text Label 6545 5555 0    60   ~ 0
+PIN_5
+Wire Wire Line
+	3660 1540 3935 1540
+Wire Wire Line
+	3935 1740 3660 1740
+Text Label 3660 1740 0    60   ~ 0
+PIN_36
+Text Label 3660 1540 0    60   ~ 0
+PIN_35
+Wire Wire Line
+	6955 5470 6955 5555
+Wire Wire Line
+	6955 5555 6545 5555
+Connection ~ 6955 5470
+Text Notes 2320 3065 0    60   ~ 0
+SPI_FLASH
+Wire Notes Line
+	3255 3065 2330 3065
 $EndSCHEMATC

Commit message: Added files via upload
Parts:
- removed SW?: SW_PUSH, symbol SW_PUSH
- added BTN?: Reset, symbol Reset
- C101: renamed from C?; footprint (none) -> Capacitors_SMD:C_0402
- J10: footprint (none) -> WIFIRE:CONN_J10
- J7: footprint (none) -> WIFIRE:CONN_J7
- J8: footprint (none) -> WIFIRE:CONN_J8
- J9: footprint (none) -> WIFIRE:CONN_J9
- JP101: renamed from JP?; footprint (none) -> Connect:PINHEAD1-3
- R101, R102, R103, R104, R105, R106, R107, R108, R109, R110: renamed from R?; footprint (none) -> Resistors_SMD:R_0402
- S101, S102, S103, S104: renamed from S?; footprint (none) -> WIFIRE:CONN_servo
- UD1: footprint (none) -> WIFIRE:HC-SR04
- j6: footprint (none) -> WIFIRE:CONN_J6
- gave numbers to parts that had none: 2
Connections:
- net GND: now also BTN?.3, BTN?.4
- net at J9.3 (P32_RST): now also BTN?.1, BTN?.2
