File: project/НИРС.sch (KiCad schematic (older format))
At the start: 26 parts, among them IC101 AT24C64A-10PU-2.7, J10 J10, J7 J7, J8 J8, J9 J9, j6 J6

Commit message: Add files via upload
Parts:
- removed R101, R102, R103, R104, R105, R106, R107, R108: 4,7K, Resistors_SMD:R_0402, symbol R
- added BTN1, BTN2, BTN3, BTN4: Button, WIFIRE:BUTTON, symbol Reset
- added D1: LED, LEDs:LED_0805, symbol LED
- added R111, R114, R115, R118, R119: 220, Resistors_SMD:R_0805, symbol R
- added R112, R113, R116, R117: 10K, Resistors_SMD:R_0805, symbol R
- C101: footprint Capacitors_SMD:C_0402 -> Capacitors_SMD:C_0805
- R109, R110: footprint Resistors_SMD:R_0402 -> Resistors_SMD:R_0805
Connections:
- net COL1 is gone; now on net LED/COL1: J10.2 (26)
- net COL2 is gone; now on net LED/COL2: J10.4 (27)
- net COL3 is gone; now on net LED/COL3: J10.6 (28)
- net COL4 is gone; now on net LED/COL4: J10.8 (29)
- net COL5 is gone; now on net LED/COL5: J10.10 (30)
- net COL6 is gone; now on net LED/COL6: J10.12 (31)
- net COL7 is gone; now on net LED/COL7: J10.14 (32)
- net COL8 is gone; now on net LED/COL8: J10.16 (33)
- net +3V3: now also R112.1, R113.1, R116.1, R117.1
- net GND: now also D1.1 (K), R114.2, R115.2, R118.2, R119.2
- net at J7.1 (8): now also R111.1
- net BTN_4: now reaches J7.10 (38)
- net BTN_4: now also BTN4.1, BTN4.2, R117.2
- net BTN_3: now reaches J7.2 (34)
- net BTN_3: now also BTN3.1, BTN3.2, R116.2
- net BTN_1: now reaches J10.5 (2)
- net BTN_1: now also BTN1.1, BTN1.2, R112.2
- net BTN_2: now reaches J8.7 (A3)
- net BTN_2: now also BTN2.1, BTN2.2, R113.2
- new net: D1.2 (A), R111.2
- new net: BTN1.3, BTN1.4, R114.1
- new net: BTN3.3, BTN3.4, R118.1
- new net: BTN2.3, BTN2.4, R115.1
- new net: BTN4.3, BTN4.4, R119.1
- no-connect marks 16 -> 11
Other:
- moved on the sheet: J10A, UD1

Commit message: Add files via upload
Parts:
- removed BTN101: Reset, WIFIRE:RESET, symbol Reset
- added A101: ADXL345, WIFIRE:ADXL345, symbol ADXL345
- added C102: 10uF, Capacitors_SMD:C_0805, symbol C
- added R102: 4.7k, Resistors_SMD:R_0805, symbol R
- added R104: 4.7K, Resistors_SMD:R_0805, symbol R
- IC101: footprint Housings_DIP:DIP-8_W7.62mm -> WIFIRE:JEDEC_SOIC
- UD1: footprint WIFIRE:HC-SR04 -> Pin_Headers:Pin_Header_Straight_1x04
Connections:
- net +3V3: now also IC101.8 (VCC), R109.2, R110.2, A101.1 (Vdd), R102.1
- net +5V: no longer IC101.8 (VCC), R109.2, R110.2
- net BTN_1: now also J10.3 (1); no longer J10.5 (2)
- net GND: now also A101.2 (GND), A101.4 (GND), A101.5 (GND), C102.1, R104.1
- net at R111.1: now also J7.12 (39); no longer J7.1 (8)
- net SDA: now reaches IC101.5 (SDA), R109.1, j6.1 (SDA)
- net SDA: now also A101.13 (SDA/SDI/SDIO)
- net SCL: now reaches IC101.6 (SCL), R110.1, j6.2 (SCL)
- net SCL: now also A101.14 (SCL/SCLK)
- new net: A101.12 (SDO/ALT_ADRESS), R104.2
- new net: A101.6 (Vs), C102.2
- new net: A101.7 (CS), R102.2
- new net INT_1: A101.8 (INT1), J10.5 (2)
- new net INT_2: A101.9 (INT2), J7.1 (8)
- no-connect marks 11 -> 13
Other:
- moved on the sheet: BTN1, BTN2, BTN3, BTN4, C101, D1, FLASH101, G1, IC101, J10A, J7, J8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
