File: project/_saved_НИРС.sch (KiCad schematic (older format))
At the start: 26 parts, among them IC101 AT24C64A-10PU-2.7, J10 J10, J7 J7, J8 J8, J9 J9, j6 J6

Commit message: Added files via upload
Parts:
- renumbered FLASH101 to FLASH, G1 to IR, UD1 to UD, IC101 to eeprom
Other:
- moved on the sheet: C101, IR, J8
Changed lines of the file:
@@
 $EndComp
 $Comp
-L AT24C64A-10PU-2.7 IC101
+L AT24C64A-10PU-2.7 eeprom
 U 1 1 56E45277
 P 9955 3200
-F 0 "IC101" H 9755 3450 50  0000 C CNN
+F 0 "eeprom" H 9755 3450 50  0000 C CNN
 F 1 "AT24C64A-10PU-2.7" H 10385 3455 50  0000 C CNN
 F 2 "Housings_DIP:DIP-8_W7.62mm" H 9330 2900 50  0001 C CIN
@@
 L J8 J8
 U 1 1 56E46A03
-P 2000 6025
-F 0 "J8" H 2000 6005 60  0000 C CNN
-F 1 "J8" H 2000 4970 60  0000 C CNN
-F 2 "WIFIRE:CONN_J8" H 2000 6025 60  0001 C CNN
-F 3 "" H 2000 6025 60  0000 C CNN
-	1    2000 6025
+P 1735 6040
+F 0 "J8" H 1735 6020 60  0000 C CNN
+F 1 "J8" H 1735 4985 60  0000 C CNN
+F 2 "WIFIRE:CONN_J8" H 1735 6040 60  0001 C CNN
+F 3 "" H 1735 6040 60  0000 C CNN
+	1    1735 6040
 	-1   0    0    1
 $EndComp
@@
 $EndComp
 $Comp
-L GP2Y0A21YK G1
+L GP2Y0A21YK IR
 U 1 1 56E4CC54
-P 1570 5720
-F 0 "G1" H 1570 5920 50  0000 C CNN
-F 1 "GP2Y0A21YK" V 1670 5720 50  0000 C CNN
-F 2 "Connect:PINHEAD1-3" V 1770 5695 50  0001 C CNN
-F 3 "" H 1570 5720 50  0000 C CNN
-	1    1570 5720
+P 1305 5735
+F 0 "IR" H 1305 5935 50  0000 C CNN
+F 1 "GP2Y0A21YK" V 1405 5735 50  0000 C CNN
+F 2 "Connect:PINHEAD1-3" V 1505 5710 50  0001 C CNN
+F 3 "" H 1305 5735 50  0000 C CNN
+	1    1305 5735
 	1    0    0    1
 $EndComp
@@
 L C C101
 U 1 1 56E4CE49
-P 1080 5570
-F 0 "C101" H 1105 5670 50  0000 L CNN
-F 1 "10uF" H 1105 5470 50  0000 L CNN
-F 2 "Capacitors_SMD:C_0402" H 1118 5420 50  0001 C CNN
-F 3 "" H 1080 5570 50  0000 C CNN
-	1    1080 5570
+P 815 5585
+F 0 "C101" H 840 5685 50  0000 L CNN
+F 1 "10uF" H 840 5485 50  0000 L CNN
+F 2 "Capacitors_SMD:C_0402" H 853 5435 50  0001 C CNN
+F 3 "" H 815 5585 50  0000 C CNN
+	1    815  5585
 	1    0    0    1
 $EndComp
@@
 L GND #PWR05
 U 1 1 56E4D720
-P 920 5720
-F 0 "#PWR05" H 920 5470 50  0001 C CNN
-F 1 "GND" H 920 5570 50  0000 C CNN
-F 2 "" H 920 5720 50  0000 C CNN
-F 3 "" H 920 5720 50  0000 C CNN
-	1    920  5720
+P 655 5735
+F 0 "#PWR05" H 655 5485 50  0001 C CNN
+F 1 "GND" H 655 5585 50  0000 C CNN
+F 2 "" H 655 5735 50  0000 C CNN
+F 3 "" H 655 5735 50  0000 C CNN
+	1    655  5735
 	1    0    0    -1
 $EndComp
@@
 L +5V #PWR06
 U 1 1 56E4D865
-P 920 5420
-F 0 "#PWR06" H 920 5270 50  0001 C CNN
-F 1 "+5V" H 920 5560 50  0000 C CNN
-F 2 "" H 920 5420 50  0000 C CNN
-F 3 "" H 920 5420 50  0000 C CNN
-	1    920  5420
+P 655 5435
+F 0 "#PWR06" H 655 5285 50  0001 C CNN
+F 1 "+5V" H 655 5575 50  0000 C CNN
+F 2 "" H 655 5435 50  0000 C CNN
+F 3 "" H 655 5435 50  0000 C CNN
+	1    655  5435
 	-1   0    0    -1
 $EndComp
 $Comp
-L HC-SR04 UD1
+L HC-SR04 UD
 U 1 1 56E5E261
 P 8325 4760
-F 0 "UD1" H 8325 5010 50  0000 C CNN
+F 0 "UD" H 8325 5010 50  0000 C CNN
 F 1 "HC-SR04" V 8580 4755 50  0000 C CNN
 F 2 "WIFIRE:HC-SR04" H 8325 4760 50  0001 C CNN
@@
 Text Label 3685 1940 0    60   ~ 0
 Trig
-Text Label 1125 5820 0    60   ~ 0
+Text Label 860  5835 0    60   ~ 0
 J8_A2
-Text Label 2565 5585 2    60   ~ 0
+Text Label 2300 5600 2    60   ~ 0
 J8_A2
 $Comp
@@
 	-1   0    0    -1
 $EndComp
-Text Notes 835  5225 0    60   ~ 0
+Text Notes 570  5240 0    60   ~ 0
 ИК-Дальномер
 Text Notes 8805 4395 2    60   ~ 0
@@
 $EndSheet
 $Sheet
-S 2590 4945 1235 1025
+S 2325 4960 1235 1025
 U 5702498F
 F0 "LED" 60
 F1 "file5702498E.sch" 60
-F2 "ROW1" I L 2590 5060 60
-F3 "ROW7" I L 2590 5210 60
-F4 "ROW2" I L 2590 5360 60
-F5 "ROW5" I L 2590 5510 60
-F6 "ROW3" I L 2590 5660 60
-F7 "ROW8" I L 2590 5735 60
-F8 "ROW4" I L 2590 5810 60
-F9 "ROW6" I L 2590 5885 60
-F10 "COL1" I R 3825 5060 60
-F11 "COL2" I R 3825 5190 60
-F12 "COL3" I R 3825 5300 60
-F13 "COL4" I R 3825 5430 60
-F14 "COL5" I R 3825 5550 60
-F15 "COL6" I R 3825 5680 60
-F16 "COL7" I R 3825 5820 60
-F17 "COL8" I R 3825 5910 60
+F2 "ROW1" I L 2325 5075 60
+F3 "ROW7" I L 2325 5225 60
+F4 "ROW2" I L 2325 5375 60
+F5 "ROW5" I L 2325 5525 60
+F6 "ROW3" I L 2325 5675 60
+F7 "ROW8" I L 2325 5750 60
+F8 "ROW4" I L 2325 5825 60
+F9 "ROW6" I L 2325 5900 60
+F10 "COL1" I R 3560 5075 60
+F11 "COL2" I R 3560 5205 60
+F12 "COL3" I R 3560 5315 60
+F13 "COL4" I R 3560 5445 60
+F14 "COL5" I R 3560 5565 60
+F15 "COL6" I R 3560 5695 60
+F16 "COL7" I R 3560 5835 60
+F17 "COL8" I R 3560 5925 60
 $EndSheet
 $Comp
@@
 Vin
 Text Label 6590 2085 0    60   ~ 0
-PWR
-Text Label 5420 1650 0    60   ~ 0
 PWR
 $Comp
@@
 	1    0    0    -1
 $EndComp
-Text Label 7395 1700 0    60   ~ 0
-PWR
 $Comp
 L GND #PWR014
@@
 Text Label 7395 2220 0    60   ~ 0
 PWM4
-Text HLabel 4330 5970 0    60   Input ~ 0
-COL8
-Text HLabel 4665 5770 0    60   Input ~ 0
-COL7
-Text HLabel 4995 5570 0    60   Input ~ 0
-COL6
-Text HLabel 5325 5370 0    60   Input ~ 0
-COL5
-Text HLabel 5655 5170 0    60   Input ~ 0
-COL4
-Text HLabel 5985 4970 0    60   Input ~ 0
-COL3
-Text HLabel 6315 4770 0    60   Input ~ 0
-COL2
-Text HLabel 6645 4570 0    60   Input ~ 0
-COL1
-$Comp
-L W25Q32BV FLASH101
+$Comp
+L W25Q32BV FLASH
 U 1 1 5709C5FC
 P 3180 3430
-F 0 "FLASH101" H 3205 2930 60  0000 C CNN
+F 0 "FLASH" H 3205 2930 60  0000 C CNN
 F 1 "W25Q32BV" H 3180 3480 60  0000 C CNN
 F 2 "WIFIRE:SOIC-8(.208mil)" H 3180 2930 60  0001 C CNN
@@
 $EndComp
 Wire Notes Line
-	1700 5240 840  5240
+	1435 5255 575  5255
 Wire Notes Line
-	1700 5960 1700 5240
+	1435 5975 1435 5255
 Wire Notes Line
 	10870 2670 10870 3870
@@
 Wire Wire Line
 	8525 4810 8795 4810
-Connection ~ 1080 5420
-Connection ~ 1080 5720
-Wire Wire Line
-	920  5420 1295 5420
-Wire Wire Line
-	1295 5420 1295 5620
-Wire Wire Line
-	1295 5620 1370 5620
-Wire Wire Line
-	920  5720 1370 5720
+Connection ~ 815  5435
+Connection ~ 815  5735
+Wire Wire Line
+	655  5435 1030 5435
+Wire Wire Line
+	1030 5435 1030 5635
+Wire Wire Line
+	1030 5635 1105 5635
+Wire Wire Line
+	655  5735 1105 5735
 Wire Wire Line
 	10755 3225 10800 3225
@@
 	7040 5870 6790 5870
 Wire Wire Line
-	6645 4570 7040 4570
-Wire Wire Line
-	6315 4770 7040 4770
-Wire Wire Line
-	5985 4970 7040 4970
-Wire Wire Line
-	5655 5170 7040 5170
-Wire Wire Line
-	4665 5770 7040 5770
+	6405 4570 7040 4570
+Wire Wire Line
+	6075 4770 7040 4770
+Wire Wire Line
+	5745 4970 7040 4970
+Wire Wire Line
+	5415 5170 7040 5170
+Wire Wire Line
+	4425 5770 7040 5770
 Wire Wire Line
 	9575 1800 9775 1800
@@
 	3935 1440 3660 1440
 Wire Wire Line
-	5325 5370 7040 5370
-Wire Wire Line
-	4995 5570 7040 5570
+	5085 5370 7040 5370
+Wire Wire Line
+	4755 5570 7040 5570
 Wire Wire Line
 	6670 4480 6670 4570
@@
 	8035 4395 8035 5055
 Wire Wire Line
-	1370 5820 1125 5820
+	1105 5835 860  5835
 Wire Wire Line
 	9575 1900 9665 1900
@@
 	10355 3715 10440 3715
 Wire Wire Line
-	2315 5885 2590 5885
-Wire Wire Line
-	2315 5735 2590 5735
-Wire Wire Line
-	2315 5585 2565 5585
-Wire Wire Line
-	2315 5810 2590 5810
-Wire Wire Line
-	2315 5660 2590 5660
-Wire Wire Line
-	2315 5510 2590 5510
+	2050 5900 2325 5900
+Wire Wire Line
+	2050 5750 2325 5750
+Wire Wire Line
+	2050 5600 2300 5600
+Wire Wire Line
+	2050 5825 2325 5825
+Wire Wire Line
+	2050 5675 2325 5675
+Wire Wire Line
+	2050 5525 2325 5525
 Wire Wire Line
 	9775 1800 9775 1995
 Wire Wire Line
-	2315 5060 2590 5060
-Wire Wire Line
-	2315 5360 2590 5360
-Wire Wire Line
-	2315 5210 2590 5210
+	2050 5075 2325 5075
+Wire Wire Line
+	2050 5375 2325 5375
+Wire Wire Line
+	2050 5225 2325 5225
 Wire Wire Line
 	4360 5970 4360 4480
@@
 	6820 2085 6590 2085
 Wire Wire Line
-	5670 1650 5420 1650
-Wire Wire Line
 	5670 1755 5630 1755
 Wire Wire Line
@@
 	7645 2220 7395 2220
 Wire Wire Line
-	4330 5970 7040 5970
+	4090 5970 7040 5970
 Wire Wire Line
 	7040 5270 6790 5270
@@
 	10356 1050 10356 1250
 Connection ~ 10356 1250
-NoConn ~ 2315 5435
-NoConn ~ 2315 5285
-NoConn ~ 2315 5135
+NoConn ~ 2050 5450
+NoConn ~ 2050 5300
+NoConn ~ 2050 5150
 NoConn ~ 7040 4870
 NoConn ~ 7040 4670
@@
 Connection ~ 9665 1800
 NoConn ~ 9575 1400
-Wire Wire Line
-	7645 1700 7395 1700
 NoConn ~ 3935 2740
 NoConn ~ 3935 2640
@@
 NoConn ~ 3935 1340
 NoConn ~ 3935 1240
+Text Label 7415 1700 0    60   ~ 0
+PWR
+Wire Wire Line
+	7645 1700 7415 1700
+Text Label 5440 1650 0    60   ~ 0
+PWR
+Wire Wire Line
+	5670 1650 5440 1650
+Text Label 3800 5075 2    60   ~ 0
+COL1
+Wire Wire Line
+	3560 5075 3800 5075
+Text Label 3800 5205 2    60   ~ 0
+COL2
+Wire Wire Line
+	3560 5205 3800 5205
+Text Label 3800 5315 2    60   ~ 0
+COL3
+Wire Wire Line
+	3560 5315 3800 5315
+Text Label 3800 5445 2    60   ~ 0
+COL4
+Wire Wire Line
+	3560 5445 3800 5445
+Text Label 3800 5565 2    60   ~ 0
+COL5
+Wire Wire Line
+	3560 5565 3800 5565
+Text Label 3800 5695 2    60   ~ 0
+COL6
+Wire Wire Line
+	3560 5695 3800 5695
+Text Label 3800 5835 2    60   ~ 0
+COL7
+Wire Wire Line
+	3560 5835 3800 5835
+Text Label 3800 5925 2    60   ~ 0
+COL8
+Wire Wire Line
+	3560 5925 3800 5925
+Text Label 6405 4570 0    60   ~ 0
+COL1
+Text Label 6075 4770 0    60   ~ 0
+COL2
+Text Label 5745 4970 0    60   ~ 0
+COL3
+Text Label 5415 5170 0    60   ~ 0
+COL4
+Text Label 5085 5370 0    60   ~ 0
+COL5
+Text Label 4755 5570 0    60   ~ 0
+COL6
+Text Label 4425 5770 0    60   ~ 0
+COL7
+Text Label 4090 5970 0    60   ~ 0
+COL8
 $EndSCHEMATC

Commit message: Added files via upload
Parts:
- BTN101: footprint WIFIRE:RESET -> WIFIRE:TS-A2PS-130
- renumbered FLASH to FLASH101, IR to G1, eeprom to IC101, UD to UD1
Other:
- moved on the sheet: C101, G1, J8
Changed lines of the file:
@@
 LIBS:valves
 LIBS:WIFIRE
+LIBS:spiflash_16m
 LIBS:НИРС-cache
 EELAYER 25 0
@@
 $EndComp
 $Comp
-L AT24C64A-10PU-2.7 eeprom
+L AT24C64A-10PU-2.7 IC101
 U 1 1 56E45277
 P 9955 3200
-F 0 "eeprom" H 9755 3450 50  0000 C CNN
+F 0 "IC101" H 9755 3450 50  0000 C CNN
 F 1 "AT24C64A-10PU-2.7" H 10385 3455 50  0000 C CNN
 F 2 "Housings_DIP:DIP-8_W7.62mm" H 9330 2900 50  0001 C CIN
@@
 L J8 J8
 U 1 1 56E46A03
-P 1735 6040
-F 0 "J8" H 1735 6020 60  0000 C CNN
-F 1 "J8" H 1735 4985 60  0000 C CNN
-F 2 "WIFIRE:CONN_J8" H 1735 6040 60  0001 C CNN
-F 3 "" H 1735 6040 60  0000 C CNN
-	1    1735 6040
+P 2000 6025
+F 0 "J8" H 2000 6005 60  0000 C CNN
+F 1 "J8" H 2000 4970 60  0000 C CNN
+F 2 "WIFIRE:CONN_J8" H 2000 6025 60  0001 C CNN
+F 3 "" H 2000 6025 60  0000 C CNN
+	1    2000 6025
 	-1   0    0    1
 $EndComp
@@
 $EndComp
 $Comp
-L GP2Y0A21YK IR
+L GP2Y0A21YK G1
 U 1 1 56E4CC54
-P 1305 5735
-F 0 "IR" H 1305 5935 50  0000 C CNN
-F 1 "GP2Y0A21YK" V 1405 5735 50  0000 C CNN
-F 2 "Connect:PINHEAD1-3" V 1505 5710 50  0001 C CNN
-F 3 "" H 1305 5735 50  0000 C CNN
-	1    1305 5735
+P 1570 5720
+F 0 "G1" H 1570 5920 50  0000 C CNN
+F 1 "GP2Y0A21YK" V 1670 5720 50  0000 C CNN
+F 2 "Connect:PINHEAD1-3" V 1770 5695 50  0001 C CNN
+F 3 "" H 1570 5720 50  0000 C CNN
+	1    1570 5720
 	1    0    0    1
 $EndComp
@@
 L C C101
 U 1 1 56E4CE49
-P 815 5585
-F 0 "C101" H 840 5685 50  0000 L CNN
-F 1 "10uF" H 840 5485 50  0000 L CNN
-F 2 "Capacitors_SMD:C_0402" H 853 5435 50  0001 C CNN
-F 3 "" H 815 5585 50  0000 C CNN
-	1    815  5585
+P 1080 5570
+F 0 "C101" H 1105 5670 50  0000 L CNN
+F 1 "10uF" H 1105 5470 50  0000 L CNN
+F 2 "Capacitors_SMD:C_0402" H 1118 5420 50  0001 C CNN
+F 3 "" H 1080 5570 50  0000 C CNN
+	1    1080 5570
 	1    0    0    1
 $EndComp
@@
 L GND #PWR05
 U 1 1 56E4D720
-P 655 5735
-F 0 "#PWR05" H 655 5485 50  0001 C CNN
-F 1 "GND" H 655 5585 50  0000 C CNN
-F 2 "" H 655 5735 50  0000 C CNN
-F 3 "" H 655 5735 50  0000 C CNN
-	1    655  5735
+P 920 5720
+F 0 "#PWR05" H 920 5470 50  0001 C CNN
+F 1 "GND" H 920 5570 50  0000 C CNN
+F 2 "" H 920 5720 50  0000 C CNN
+F 3 "" H 920 5720 50  0000 C CNN
+	1    920  5720
 	1    0    0    -1
 $EndComp
@@
 L +5V #PWR06
 U 1 1 56E4D865
-P 655 5435
-F 0 "#PWR06" H 655 5285 50  0001 C CNN
-F 1 "+5V" H 655 5575 50  0000 C CNN
-F 2 "" H 655 5435 50  0000 C CNN
-F 3 "" H 655 5435 50  0000 C CNN
-	1    655  5435
+P 920 5420
+F 0 "#PWR06" H 920 5270 50  0001 C CNN
+F 1 "+5V" H 920 5560 50  0000 C CNN
+F 2 "" H 920 5420 50  0000 C CNN
+F 3 "" H 920 5420 50  0000 C CNN
+	1    920  5420
 	-1   0    0    -1
 $EndComp
 $Comp
-L HC-SR04 UD
+L HC-SR04 UD1
 U 1 1 56E5E261
 P 8325 4760
-F 0 "UD" H 8325 5010 50  0000 C CNN
+F 0 "UD1" H 8325 5010 50  0000 C CNN
 F 1 "HC-SR04" V 8580 4755 50  0000 C CNN
 F 2 "WIFIRE:HC-SR04" H 8325 4760 50  0001 C CNN
@@
 Text Label 3685 1940 0    60   ~ 0
 Trig
-Text Label 860  5835 0    60   ~ 0
+Text Label 1125 5820 0    60   ~ 0
 J8_A2
-Text Label 2300 5600 2    60   ~ 0
+Text Label 2565 5585 2    60   ~ 0
 J8_A2
 $Comp
@@
 	-1   0    0    -1
 $EndComp
-Text Notes 570  5240 0    60   ~ 0
+Text Notes 835  5225 0    60   ~ 0
 ИК-Дальномер
 Text Notes 8805 4395 2    60   ~ 0
@@
 $EndSheet
 $Sheet
-S 2325 4960 1235 1025
+S 2590 4945 1235 1025
 U 5702498F
 F0 "LED" 60
 F1 "file5702498E.sch" 60
-F2 "ROW1" I L 2325 5075 60
-F3 "ROW7" I L 2325 5225 60
-F4 "ROW2" I L 2325 5375 60
-F5 "ROW5" I L 2325 5525 60
-F6 "ROW3" I L 2325 5675 60
-F7 "ROW8" I L 2325 5750 60
-F8 "ROW4" I L 2325 5825 60
-F9 "ROW6" I L 2325 5900 60
-F10 "COL1" I R 3560 5075 60
-F11 "COL2" I R 3560 5205 60
-F12 "COL3" I R 3560 5315 60
-F13 "COL4" I R 3560 5445 60
-F14 "COL5" I R 3560 5565 60
-F15 "COL6" I R 3560 5695 60
-F16 "COL7" I R 3560 5835 60
-F17 "COL8" I R 3560 5925 60
+F2 "ROW1" I L 2590 5060 60
+F3 "ROW7" I L 2590 5210 60
+F4 "ROW2" I L 2590 5360 60
+F5 "ROW5" I L 2590 5510 60
+F6 "ROW3" I L 2590 5660 60
+F7 "ROW8" I L 2590 5735 60
+F8 "ROW4" I L 2590 5810 60
+F9 "ROW6" I L 2590 5885 60
+F10 "COL1" I R 3825 5060 60
+F11 "COL2" I R 3825 5190 60
+F12 "COL3" I R 3825 5300 60
+F13 "COL4" I R 3825 5430 60
+F14 "COL5" I R 3825 5550 60
+F15 "COL6" I R 3825 5680 60
+F16 "COL7" I R 3825 5820 60
+F17 "COL8" I R 3825 5910 60
 $EndSheet
 $Comp
@@
 Vin
 Text Label 6590 2085 0    60   ~ 0
+PWR
+Text Label 5420 1650 0    60   ~ 0
 PWR
 $Comp
@@
 	1    0    0    -1
 $EndComp
+Text Label 7395 1700 0    60   ~ 0
+PWR
 $Comp
 L GND #PWR014
@@
 Text Label 7395 2220 0    60   ~ 0
 PWM4
-$Comp
-L W25Q32BV FLASH
+Text HLabel 4330 5970 0    60   Input ~ 0
+COL8
+Text HLabel 4665 5770 0    60   Input ~ 0
+COL7
+Text HLabel 4995 5570 0    60   Input ~ 0
+COL6
+Text HLabel 5325 5370 0    60   Input ~ 0
+COL5
+Text HLabel 5655 5170 0    60   Input ~ 0
+COL4
+Text HLabel 5985 4970 0    60   Input ~ 0
+COL3
+Text HLabel 6315 4770 0    60   Input ~ 0
+COL2
+Text HLabel 6645 4570 0    60   Input ~ 0
+COL1
+$Comp
+L W25Q32BV FLASH101
 U 1 1 5709C5FC
 P 3180 3430
-F 0 "FLASH" H 3205 2930 60  0000 C CNN
+F 0 "FLASH101" H 3205 2930 60  0000 C CNN
 F 1 "W25Q32BV" H 3180 3480 60  0000 C CNN
 F 2 "WIFIRE:SOIC-8(.208mil)" H 3180 2930 60  0001 C CNN
@@
 F 0 "BTN101" H 10116 995 60  0000 C CNN
 F 1 "Reset" H 10116 1375 60  0000 C CNN
-F 2 "WIFIRE:RESET" H 10116 995 60  0001 C CNN
+F 2 "WIFIRE:TS-A2PS-130" H 10116 995 60  0001 C CNN
 F 3 "" H 10116 995 60  0000 C CNN
 	1    10116 1150
@@
 $EndComp
 Wire Notes Line
-	1435 5255 575  5255
+	1700 5240 840  5240
 Wire Notes Line
-	1435 5975 1435 5255
+	1700 5960 1700 5240
 Wire Notes Line
 	10870 2670 10870 3870
@@
 Wire Wire Line
 	8525 4810 8795 4810
-Connection ~ 815  5435
-Connection ~ 815  5735
-Wire Wire Line
-	655  5435 1030 5435
-Wire Wire Line
-	1030 5435 1030 5635
-Wire Wire Line
-	1030 5635 1105 5635
-Wire Wire Line
-	655  5735 1105 5735
+Connection ~ 1080 5420
+Connection ~ 1080 5720
+Wire Wire Line
+	920  5420 1295 5420
+Wire Wire Line
+	1295 5420 1295 5620
+Wire Wire Line
+	1295 5620 1370 5620
+Wire Wire Line
+	920  5720 1370 5720
 Wire Wire Line
 	10755 3225 10800 3225
@@
 	7040 5870 6790 5870
 Wire Wire Line
-	6405 4570 7040 4570
-Wire Wire Line
-	6075 4770 7040 4770
-Wire Wire Line
-	5745 4970 7040 4970
-Wire Wire Line
-	5415 5170 7040 5170
-Wire Wire Line
-	4425 5770 7040 5770
+	6645 4570 7040 4570
+Wire Wire Line
+	6315 4770 7040 4770
+Wire Wire Line
+	5985 4970 7040 4970
+Wire Wire Line
+	5655 5170 7040 5170
+Wire Wire Line
+	4665 5770 7040 5770
 Wire Wire Line
 	9575 1800 9775 1800
@@
 	3935 1440 3660 1440
 Wire Wire Line
-	5085 5370 7040 5370
-Wire Wire Line
-	4755 5570 7040 5570
+	5325 5370 7040 5370
+Wire Wire Line
+	4995 5570 7040 5570
 Wire Wire Line
 	6670 4480 6670 4570
@@
 	8035 4395 8035 5055
 Wire Wire Line
-	1105 5835 860  5835
+	1370 5820 1125 5820
 Wire Wire Line
 	9575 1900 9665 1900
@@
 	10355 3715 10440 3715
 Wire Wire Line
-	2050 5900 2325 5900
-Wire Wire Line
-	2050 5750 2325 5750
-Wire Wire Line
-	2050 5600 2300 5600
-Wire Wire Line
-	2050 5825 2325 5825
-Wire Wire Line
-	2050 5675 2325 5675
-Wire Wire Line
-	2050 5525 2325 5525
+	2315 5885 2590 5885
+Wire Wire Line
+	2315 5735 2590 5735
+Wire Wire Line
+	2315 5585 2565 5585
+Wire Wire Line
+	2315 5810 2590 5810
+Wire Wire Line
+	2315 5660 2590 5660
+Wire Wire Line
+	2315 5510 2590 5510
 Wire Wire Line
 	9775 1800 9775 1995
 Wire Wire Line
-	2050 5075 2325 5075
-Wire Wire Line
-	2050 5375 2325 5375
-Wire Wire Line
-	2050 5225 2325 5225
+	2315 5060 2590 5060
+Wire Wire Line
+	2315 5360 2590 5360
+Wire Wire Line
+	2315 5210 2590 5210
 Wire Wire Line
 	4360 5970 4360 4480
@@
 	6820 2085 6590 2085
 Wire Wire Line
+	5670 1650 5420 1650
+Wire Wire Line
 	5670 1755 5630 1755
 Wire Wire Line
@@
 	7645 2220 7395 2220
 Wire Wire Line
-	4090 5970 7040 5970
+	4330 5970 7040 5970
 Wire Wire Line
 	7040 5270 6790 5270
@@
 	10356 1050 10356 1250
 Connection ~ 10356 1250
-NoConn ~ 2050 5450
-NoConn ~ 2050 5300
-NoConn ~ 2050 5150
+NoConn ~ 2315 5435
+NoConn ~ 2315 5285
+NoConn ~ 2315 5135
 NoConn ~ 7040 4870
 NoConn ~ 7040 4670
@@
 Connection ~ 9665 1800
 NoConn ~ 9575 1400
+Wire Wire Line
+	7645 1700 7395 1700
 NoConn ~ 3935 2740
 NoConn ~ 3935 2640
@@
 NoConn ~ 3935 1340
 NoConn ~ 3935 1240
-Text Label 7415 1700 0    60   ~ 0
-PWR
-Wire Wire Line
-	7645 1700 7415 1700
-Text Label 5440 1650 0    60   ~ 0
-PWR
-Wire Wire Line
-	5670 1650 5440 1650
-Text Label 3800 5075 2    60   ~ 0
-COL1
-Wire Wire Line
-	3560 5075 3800 5075
-Text Label 3800 5205 2    60   ~ 0
-COL2
-Wire Wire Line
-	3560 5205 3800 5205
-Text Label 3800 5315 2    60   ~ 0
-COL3
-Wire Wire Line
-	3560 5315 3800 5315
-Text Label 3800 5445 2    60   ~ 0
-COL4
-Wire Wire Line
-	3560 5445 3800 5445
-Text Label 3800 5565 2    60   ~ 0
-COL5
-Wire Wire Line
-	3560 5565 3800 5565
-Text Label 3800 5695 2    60   ~ 0
-COL6
-Wire Wire Line
-	3560 5695 3800 5695
-Text Label 3800 5835 2    60   ~ 0
-COL7
-Wire Wire Line
-	3560 5835 3800 5835
-Text Label 3800 5925 2    60   ~ 0
-COL8
-Wire Wire Line
-	3560 5925 3800 5925
-Text Label 6405 4570 0    60   ~ 0
-COL1
-Text Label 6075 4770 0    60   ~ 0
-COL2
-Text Label 5745 4970 0    60   ~ 0
-COL3
-Text Label 5415 5170 0    60   ~ 0
-COL4
-Text Label 5085 5370 0    60   ~ 0
-COL5
-Text Label 4755 5570 0    60   ~ 0
-COL6
-Text Label 4425 5770 0    60   ~ 0
-COL7
-Text Label 4090 5970 0    60   ~ 0
-COL8
 $EndSCHEMATC
