File: project/НИРС.kicad_pcb (KiCad board)
At the start: 2 copper layers, 88.9 x 53.3 mm, 78 parts, among them J10 J10, J7 J7, J8 J8, J9 J9, Q301 Tran_8050, Q302 Tran_8050, Q303 Tran_8050, Q304 Tran_8050, Q305 Tran_8050, Q306 Tran_8050, Q307 Tran_8050, Q308 Tran_8050, U201 74HC595, U202 74HC595, j6 J6

Commit message: Added files via upload
Parts:
- moved Q304 46.5 mm to (184.8, 114.2)
- moved R317 46.5 mm to (184.8, 117.4)
- moved R320 46.5 mm to (184.8, 110.9)
- moved R318 46.5 mm to (181.5, 114.2)
- moved FLASH 38.3 mm to (153.2, 111.4)
- moved UD 34.3 mm to (138.2, 142.1)
- moved eeprom 33.5 mm to (129.8, 106.7)
- moved R109 33.5 mm to (133.6, 109.6)
- moved R110 33.5 mm to (133.6, 112.0)
- moved R306 32.9 mm to (186.7, 132.7)
- moved R305 32.9 mm to (184.4, 132.7)
- moved R308 31.4 mm to (186.7, 135.7)
- moved R307 31.4 mm to (184.4, 135.7)
- moved R301 31.2 mm to (184.4, 126.8)
- moved R302 31.2 mm to (186.7, 126.8)
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Routing:
- net GND: track 0.00 -> 240.9 mm, vias 0 -> 28
- net +5V: track 0.00 -> 160.9 mm, vias 0 -> 20
- net /J8_A2: track 0.00 -> 98.0 mm, vias 0 -> 1
- net /Echo: track 0.00 -> 70.3 mm, vias 0 -> 6
- net /PIN_5: track 0.00 -> 69.6 mm, vias 0 -> 3
- net /Trig: track 0.00 -> 59.8 mm, vias 0 -> 7
- net /LED/COL1: track 0.00 -> 58.6 mm, vias 0 -> 4
- net /7-SEGM/RCLK: track 0.00 -> 55.9 mm, vias 0 -> 2
- net /PWR: track 0.00 -> 53.3 mm
- net /LED/COL6: track 0.00 -> 48.4 mm, vias 0 -> 4
- net +3V3: track 0.00 -> 46.7 mm
- net /7-SEGM/SRCLK: track 0.00 -> 45.0 mm, vias 0 -> 2
- net Net-(R206-Pad1): track 0.00 -> 44.4 mm, vias 0 -> 4
- net /PWM1: track 0.00 -> 42.2 mm, vias 0 -> 1
- net /LED/COL3: track 0.00 -> 41.7 mm, vias 0 -> 2
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- added copper zone on B.Cu, net GND
- added copper zone on F.Cu, net GND
Other:
- board size 88.9 x 53.3 mm -> 70.7 x 54.3 mm

Commit message: Added files via upload
Parts:
- FLASH: footprint WIFIRE:SOIC-8(.208mil) -> WIFIRE:SOIC-8(.208mil)new
- RESET: footprint WIFIRE:RESET -> WIFIRE:TS-A2PS-130
- eeprom: footprint Housings_DIP:DIP-8_W7.62mm -> WIFIRE:JEDEC_SOIC; moved to B.Cu
- moved UD 14.0 mm to (138.2, 128.1)
- moved RESET 8.36 mm to (173.6, 135.3)
- moved eeprom 6.50 mm to (133.8, 111.8)
- moved R110 4.83 mm to (138.4, 111.8), turned to 270 degrees
- moved R109 4.81 mm to (129.3, 111.8), turned to 270 degrees
- moved S101 4.00 mm to (194.1, 138.6)
- moved S104 4.00 mm to (194.1, 107.8)
- moved S102 2.00 mm to (194.1, 129.0)
- moved S103 2.00 mm to (194.1, 117.4)
Routing:
- net /PWR: track 53.3 -> 62.3 mm, vias 0 -> 1
- net /J8_A2: track 98.0 -> 89.3 mm, vias 1 -> 2
- net /PIN_5: track 69.6 -> 75.8 mm, vias 3 -> 2
- net /PWM1: track 42.2 -> 48.2 mm, vias 1 -> 0
- net /LED/COL1: track 58.6 -> 64.6 mm, vias 4 -> 5
- net /Trig: track 59.8 -> 54.4 mm, vias 7 -> 3
- net Net-(IC101-Pad6): track 29.5 -> 24.3 mm, vias 3 -> 1
- net +5V: track 160.9 -> 165.5 mm
- net Net-(IC101-Pad5): track 27.3 -> 23.4 mm, vias 2 -> 0
- net /PWM4: track 36.0 -> 32.2 mm, vias 3 -> 2
- net /LED/ROW7: track 13.0 -> 9.63 mm
- net Net-(BTN101-Pad1): track 24.6 -> 27.9 mm, vias 1 -> 0
- net /Echo: track 70.3 -> 72.8 mm, vias 6 -> 4
- net /7-SEGM/SER: track 27.9 -> 26.1 mm
- net Net-(LED301-Pad1): track 23.2 -> 21.6 mm, vias 2 -> 1
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Other:
- board size 70.7 x 54.3 mm -> 68 x 53.3 mm
- board text added: "4k7"

Commit message: Added files via upload
Parts:
- moved IR 49.2 mm to (143.6, 147.3)
- moved C101 48.1 mm to (149.8, 147.5), turned to 270 degrees
- moved eeprom 28.2 mm to (138.8, 139.6), turned to 270 degrees
- moved R110 22.9 mm to (137.0, 134.7)
- moved R109 21.2 mm to (137.0, 131.6)
- moved URM 4.96 mm to (139.0, 123.2)
- renumbered DISP201 to DISP, JP101 to JMPR, LED301 to LED, S101 to SRV1, S102 to SRV2, S103 to SRV3, S104 to SRV4, UD to URM
Routing:
- net /J8_A2: track 89.3 -> 41.7 mm, vias 2 -> 0
- net Net-(IC101-Pad5): track 23.4 -> 55.2 mm
- net Net-(IC101-Pad6): track 24.3 -> 55.6 mm
- net +5V: track 165.5 -> 187.5 mm, vias 20 -> 18
- net GND: track 240.7 -> 224.1 mm, vias 24 -> 23
- net /Echo: track 72.8 -> 77.2 mm, vias 4 -> 2
- net /Trig: track 54.4 -> 57.5 mm
- net /LED/GNM_13: track 26.7 -> 24.7 mm
- net /LED/GNM_11: track 39.8 -> 38.1 mm
- net /7-SEGM/Dig3: track 26.6 -> 27.5 mm
- net Net-(LED301-Pad5): vias 2 -> 1
- net /7-SEGM/QH: vias 2 -> 0
Other:
- board size 68 x 53.3 mm -> 60.1 x 53.3 mm
- board text added: "0 26"
- board text added: "3V3"
- board text added: "5V"
- board text added: "5V0"
- board text added: "A6 A0"
- board text added: "GND"
- board text added: "Vin"
