File: project/НИРС.kicad_pcb (KiCad board)
At the start: 2 copper layers, 62.9 x 53.3 mm, 85 parts, among them J10 J10, J7 J7, J8 J8, J9 J9, Q301 Tran_8050, Q302 Tran_8050, Q303 Tran_8050, Q304 Tran_8050, Q305 Tran_8050, Q306 Tran_8050, Q307 Tran_8050, Q308 Tran_8050, U201 74HC595, U202 74HC595, j6 J6

Commit message: Add files via upload
Parts:
- removed RESET: Reset, WIFIRE:TS-A2PS-130
- added Accel: ADXL345, WIFIRE:ADXL345, F.Cu at (161.8, 113.8)
- added C102: 10uF, Capacitors_SMD:C_0805, B.Cu at (158.6, 114.9)
- added R102: 4.7k, Resistors_SMD:R_0805, B.Cu at (158.4, 122.3)
- added R104: 4.7K, Resistors_SMD:R_0805, B.Cu at (158.4, 118.7)
- moved J7_10 35.2 mm to (182.1, 136.2), turned to 270 degrees
- moved R119 33.9 mm to (177.6, 136.3)
- moved R118 22.0 mm to (174.5, 136.2)
- moved J7_2 17.8 mm to (169.9, 136.1), turned to 90 degrees
- moved G*** 11.8 mm to (161.9, 123.0)
- moved JMPR 11.7 mm to (156.2, 144.8)
- renumbered DISP to 7-SEGM, BTN1 to J10_3, BTN4 to J7_10, BTN3 to J7_2, BTN2 to J8_7, U201 to REG_1, U202 to REG_2
Connections:
- net Net-(IC101-Pad5) renamed /SDA
- net Net-(IC101-Pad6) renamed /SCL
- J10 pad 3: Net-(J10-Pad3) -> /BTN_1
- J10 pad 5: /BTN_1 -> /INT_1
- J7 pad 1: Net-(J7-Pad1) -> /INT_2
- R109 pad 2: +5V -> +3V3
- R110 pad 2: +5V -> +3V3
- R111 pad 1: Net-(J7-Pad1) -> Net-(J7-Pad12)
- eeprom pad 8: +5V -> +3V3
Routing:
- net GND: track 827.6 -> 917.2 mm, vias 70 -> 77
- net /INT_1: track 0.00 -> 40.2 mm, vias 0 -> 6
- net +3V3: track 69.6 -> 101.7 mm
- net Net-(J9-Pad3): track 29.1 -> 0.00 mm, vias 2 -> 0
- net Net-(J7-Pad1): track 28.2 -> 0.00 mm, vias 1 -> 0
- net /BTN_4: track 44.9 -> 72.4 mm, vias 1 -> 2
- net /INT_2: track 0.00 -> 21.2 mm, vias 0 -> 3
- net +5V: track 127.6 -> 106.5 mm
- net /SCL: track 54.4 -> 70.0 mm, vias 1 -> 4
- net Net-(A101-Pad12): track 0.00 -> 13.7 mm, vias 0 -> 1
- net Net-(LED301-Pad5): track 27.2 -> 39.3 mm
- net /SDA: track 46.7 -> 58.5 mm, vias 1 -> 4
- net Net-(J7-Pad12): track 0.00 -> 11.6 mm, vias 0 -> 1
- net /PWR: track 64.0 -> 75.6 mm
- net /Vin: track 5.83 -> 13.8 mm
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Other:
- board text added: "Echo"
- board text added: "Trig"
- board text added: "Vcc"
- board text added: "Vo"
