File: project/_autosave-НИРС.kicad_pcb (KiCad board)
At the start: 2 copper layers, 62.9 x 53.3 mm, 85 parts, among them J10 J10, J7 J7, J8 J8, J9 J9, Q301 Tran_8050, Q302 Tran_8050, Q303 Tran_8050, Q304 Tran_8050, Q305 Tran_8050, Q306 Tran_8050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

Commit message: Add files via upload
Parts:
- moved JMPR 11.7 mm to (156.2, 144.8)
Routing:
- net /PWR: track 64.0 -> 76.9 mm, vias 0 -> 2
- net /Vin: track 5.83 -> 13.8 mm, vias 0 -> 1
- net +5V: track 127.6 -> 130.2 mm
- net GND: track 827.6 -> 825.4 mm
- net Net-(BTN101-Pad1): track 29.1 -> 28.1 mm
