File: project/file56F4BED3.sch (KiCad schematic (older format))
At the start: 11 parts

Commit message: Added files via upload
Parts:
- DISP201: renamed from DISP?; footprint (none) -> WIFIRE:BA56-12SRWA
- R201, R202, R203, R204, R205, R206, R207, R208: renamed from R?; footprint (none) -> Resistors_SMD:R_0402
- U201, U202: renamed from U?; footprint (none) -> Housings_SOIC:SOIC-16_3.9x9.9mm_Pitch1.27mm
Changed lines of the file:
@@
 $EndDescr
 $Comp
-L 74HC595 U?
+L 74HC595 U202
 U 1 1 56F5E43D
 P 4550 2880
-F 0 "U?" H 4700 3480 50  0000 C CNN
+F 0 "U202" H 4700 3480 50  0000 C CNN
 F 1 "74HC595" H 4550 2280 50  0000 C CNN
-F 2 "" H 4550 2880 50  0000 C CNN
+F 2 "Housings_SOIC:SOIC-16_3.9x9.9mm_Pitch1.27mm" H 4550 2880 50  0001 C CNN
 F 3 "" H 4550 2880 50  0000 C CNN
 	1    4550 2880
@@
 $EndComp
 $Comp
-L R R?
+L R R201
 U 1 1 56F5E444
 P 5460 2265
-F 0 "R?" V 5540 2265 50  0000 C CNN
+F 0 "R201" V 5540 2265 50  0000 C CNN
 F 1 "68" V 5460 2265 50  0000 C CNN
-F 2 "" V 5390 2265 50  0000 C CNN
+F 2 "Resistors_SMD:R_0402" V 5390 2265 50  0001 C CNN
 F 3 "" H 5460 2265 50  0000 C CNN
 	1    5460 2265
@@
 $EndComp
 $Comp
-L R R?
+L R R207
 U 1 1 56F5E44B
 P 5460 3195
-F 0 "R?" V 5540 3195 50  0000 C CNN
+F 0 "R207" V 5540 3195 50  0000 C CNN
 F 1 "68" V 5460 3195 50  0000 C CNN
-F 2 "" V 5390 3195 50  0000 C CNN
+F 2 "Resistors_SMD:R_0402" V 5390 3195 50  0001 C CNN
 F 3 "" H 5460 3195 50  0000 C CNN
 	1    5460 3195
@@
 $EndComp
 $Comp
-L R R?
+L R R205
 U 1 1 56F5E452
 P 5460 2885
-F 0 "R?" V 5540 2885 50  0000 C CNN
+F 0 "R205" V 5540 2885 50  0000 C CNN
 F 1 "68" V 5460 2885 50  0000 C CNN
-F 2 "" V 5390 2885 50  0000 C CNN
+F 2 "Resistors_SMD:R_0402" V 5390 2885 50  0001 C CNN
 F 3 "" H 5460 2885 50  0000 C CNN
 	1    5460 2885
@@
 $EndComp
 $Comp
-L R R?
+L R R203
 U 1 1 56F5E459
 P 5460 2575
-F 0 "R?" V 5540 2575 50  0000 C CNN
+F 0 "R203" V 5540 2575 50  0000 C CNN
 F 1 "68" V 5460 2575 50  0000 C CNN
-F 2 "" V 5390 2575 50  0000 C CNN
+F 2 "Resistors_SMD:R_0402" V 5390 2575 50  0001 C CNN
 F 3 "" H 5460 2575 50  0000 C CNN
 	1    5460 2575
@@
 $EndComp
 $Comp
-L R R?
+L R R202
 U 1 1 56F5E460
 P 5460 2420
-F 0 "R?" V 5540 2420 50  0000 C CNN
+F 0 "R202" V 5540 2420 50  0000 C CNN
 F 1 "68" V 5460 2420 50  0000 C CNN
-F 2 "" V 5390 2420 50  0000 C CNN
+F 2 "Resistors_SMD:R_0402" V 5390 2420 50  0001 C CNN
 F 3 "" H 5460 2420 50  0000 C CNN
 	1    5460 2420
@@
 $EndComp
 $Comp
-L R R?
+L R R208
 U 1 1 56F5E467
 P 5460 3350
-F 0 "R?" V 5540 3350 50  0000 C CNN
+F 0 "R208" V 5540 3350 50  0000 C CNN
 F 1 "68" V 5460 3350 50  0000 C CNN
-F 2 "" V 5390 3350 50  0000 C CNN
+F 2 "Resistors_SMD:R_0402" V 5390 3350 50  0001 C CNN
 F 3 "" H 5460 3350 50  0000 C CNN
 	1    5460 3350
@@
 $EndComp
 $Comp
-L R R?
+L R R206
 U 1 1 56F5E46E
 P 5460 3040
-F 0 "R?" V 5540 3040 50  0000 C CNN
+F 0 "R206" V 5540 3040 50  0000 C CNN
 F 1 "68" V 5460 3040 50  0000 C CNN
-F 2 "" V 5390 3040 50  0000 C CNN
+F 2 "Resistors_SMD:R_0402" V 5390 3040 50  0001 C CNN
 F 3 "" H 5460 3040 50  0000 C CNN
 	1    5460 3040
@@
 $EndComp
 $Comp
-L R R?
+L R R204
 U 1 1 56F5E475
 P 5460 2730
-F 0 "R?" V 5540 2730 50  0000 C CNN
+F 0 "R204" V 5540 2730 50  0000 C CNN
 F 1 "68" V 5460 2730 50  0000 C CNN
-F 2 "" V 5390 2730 50  0000 C CNN
+F 2 "Resistors_SMD:R_0402" V 5390 2730 50  0001 C CNN
 F 3 "" H 5460 2730 50  0000 C CNN
 	1    5460 2730
@@
 $EndComp
 $Comp
-L +5V #PWR?
+L +5V #PWR021
 U 1 1 56F5E47C
 P 3830 2375
-F 0 "#PWR?" H 3830 2225 50  0001 C CNN
+F 0 "#PWR021" H 3830 2225 50  0001 C CNN
 F 1 "+5V" H 3830 2515 50  0000 C CNN
 F 2 "" H 3830 2375 50  0000 C CNN
@@
 $EndComp
 $Comp
-L GND #PWR?
+L GND #PWR022
 U 1 1 56F5E482
 P 3675 4335
-F 0 "#PWR?" H 3675 4085 50  0001 C CNN
+F 0 "#PWR022" H 3675 4085 50  0001 C CNN
 F 1 "GND" H 3675 4185 50  0000 C CNN
 F 2 "" H 3675 4335 50  0000 C CNN
@@
 $EndComp
 $Comp
-L GND #PWR?
+L GND #PWR023
 U 1 1 56F5E488
 P 3830 3075
-F 0 "#PWR?" H 3830 2825 50  0001 C CNN
+F 0 "#PWR023" H 3830 2825 50  0001 C CNN
 F 1 "GND" H 3830 2925 50  0000 C CNN
 F 2 "" H 3830 3075 50  0000 C CNN
@@
 NoConn ~ 5225 4605
 $Comp
-L +5V #PWR?
+L +5V #PWR024
 U 1 1 56F5E494
 P 3675 3985
-F 0 "#PWR?" H 3675 3835 50  0001 C CNN
+F 0 "#PWR024" H 3675 3835 50  0001 C CNN
 F 1 "+5V" H 3675 4125 50  0000 C CNN
 F 2 "" H 3675 3985 50  0000 C CNN
@@
 $EndComp
 $Comp
-L 74HC595 U?
+L 74HC595 U201
 U 1 1 56F5E49A
 P 4525 4155
-F 0 "U?" H 4675 4755 50  0000 C CNN
+F 0 "U201" H 4675 4755 50  0000 C CNN
 F 1 "74HC595" H 4525 3555 50  0000 C CNN
-F 2 "" H 4525 4155 50  0000 C CNN
+F 2 "Housings_SOIC:SOIC-16_3.9x9.9mm_Pitch1.27mm" H 4525 4155 50  0001 C CNN
 F 3 "" H 4525 4155 50  0000 C CNN
 	1    4525 4155
@@
 QE
 $Comp
-L BA56-12SRWA(2) DISP?
+L BA56-12SRWA(2) DISP201
 U 1 1 56F5E4D5
 P 6745 2975
-F 0 "DISP?" H 7260 1890 50  0000 C CNN
+F 0 "DISP201" H 7260 1890 50  0000 C CNN
 F 1 "BA56-12SRWA(2)" H 7280 2935 50  0000 C CNN
-F 2 "" H 6335 2410 50  0000 C CNN
+F 2 "WIFIRE:BA56-12SRWA" H 6335 2410 50  0001 C CNN
 F 3 "" H 6335 2410 50  0000 C CNN
 	1    6745 2975

Commit message: Added files via upload
Connections:
- net +5V: now also U201.16 (VCC), U202.16 (VCC)
- net GND: now also U201.8 (GND), U202.8 (GND)
Other:
- moved on the sheet: U201
Changed lines of the file:
@@
 P 4550 2880
 F 0 "U202" H 4700 3480 50  0000 C CNN
-F 1 "74HC595" H 4550 2280 50  0000 C CNN
+F 1 "74HC595" H 4600 2285 50  0000 C CNN
 F 2 "Housings_SOIC:SOIC-16_3.9x9.9mm_Pitch1.27mm" H 4550 2880 50  0001 C CNN
 F 3 "" H 4550 2880 50  0000 C CNN
@@
 $EndComp
 $Comp
-L +5V #PWR021
-U 1 1 56F5E47C
-P 3830 2375
-F 0 "#PWR021" H 3830 2225 50  0001 C CNN
-F 1 "+5V" H 3830 2515 50  0000 C CNN
-F 2 "" H 3830 2375 50  0000 C CNN
-F 3 "" H 3830 2375 50  0000 C CNN
-	1    3830 2375
-	-1   0    0    -1
-$EndComp
-$Comp
 L GND #PWR022
 U 1 1 56F5E482
-P 3675 4335
-F 0 "#PWR022" H 3675 4085 50  0001 C CNN
-F 1 "GND" H 3675 4185 50  0000 C CNN
-F 2 "" H 3675 4335 50  0000 C CNN
-F 3 "" H 3675 4335 50  0000 C CNN
-	1    3675 4335
+P 4365 5055
+F 0 "#PWR022" H 4365 4805 50  0001 C CNN
+F 1 "GND" H 4365 4905 50  0000 C CNN
+F 2 "" H 4365 5055 50  0000 C CNN
+F 3 "" H 4365 5055 50  0000 C CNN
+	1    4365 5055
 	1    0    0    -1
 $EndComp
@@
 L GND #PWR023
 U 1 1 56F5E488
-P 3830 3075
-F 0 "#PWR023" H 3830 2825 50  0001 C CNN
-F 1 "GND" H 3830 2925 50  0000 C CNN
-F 2 "" H 3830 3075 50  0000 C CNN
-F 3 "" H 3830 3075 50  0000 C CNN
-	1    3830 3075
-	1    0    0    -1
-$EndComp
-NoConn ~ 5225 4005
-NoConn ~ 5225 4105
-NoConn ~ 5225 4205
-NoConn ~ 5225 4305
-NoConn ~ 5225 4405
-NoConn ~ 5225 4605
-$Comp
-L +5V #PWR024
-U 1 1 56F5E494
-P 3675 3985
-F 0 "#PWR024" H 3675 3835 50  0001 C CNN
-F 1 "+5V" H 3675 4125 50  0000 C CNN
-F 2 "" H 3675 3985 50  0000 C CNN
-F 3 "" H 3675 3985 50  0000 C CNN
-	1    3675 3985
-	1    0    0    -1
-$EndComp
+P 3830 3255
+F 0 "#PWR023" H 3830 3005 50  0001 C CNN
+F 1 "GND" H 3830 3105 50  0000 C CNN
+F 2 "" H 3830 3255 50  0000 C CNN
+F 3 "" H 3830 3255 50  0000 C CNN
+	1    3830 3255
+	1    0    0    -1
+$EndComp
+NoConn ~ 5225 4245
+NoConn ~ 5225 4345
+NoConn ~ 5225 4445
+NoConn ~ 5225 4545
+NoConn ~ 5225 4645
+NoConn ~ 5225 4845
 $Comp
 L 74HC595 U201
 U 1 1 56F5E49A
-P 4525 4155
-F 0 "U201" H 4675 4755 50  0000 C CNN
-F 1 "74HC595" H 4525 3555 50  0000 C CNN
-F 2 "Housings_SOIC:SOIC-16_3.9x9.9mm_Pitch1.27mm" H 4525 4155 50  0001 C CNN
-F 3 "" H 4525 4155 50  0000 C CNN
-	1    4525 4155
+P 4525 4395
+F 0 "U201" H 4675 4995 50  0000 C CNN
+F 1 "74HC595" H 4585 3795 50  0000 C CNN
+F 2 "Housings_SOIC:SOIC-16_3.9x9.9mm_Pitch1.27mm" H 4525 4395 50  0001 C CNN
+F 3 "" H 4525 4395 50  0000 C CNN
+	1    4525 4395
 	1    0    0    -1
 $EndComp
@@
 Text Label 6340 2485 0    60   ~ 0
 Dig3
-Text Label 5430 3905 2    60   ~ 0
+Text Label 5430 4145 2    60   ~ 0
 Dig3
 Text Label 6340 2580 0    60   ~ 0
 Dig2
-Text Label 5430 3805 2    60   ~ 0
+Text Label 5430 4045 2    60   ~ 0
 Dig2
-Text Label 5430 3705 2    60   ~ 0
+Text Label 5430 3945 2    60   ~ 0
 Dig1
 Text Label 6340 2850 0    60   ~ 0
@@
 RCLK
 Wire Wire Line
-	3555 2930 3850 2930
+	3555 2930 3605 2930
+Wire Wire Line
+	3605 2930 3850 2930
 Connection ~ 3755 2630
 Wire Wire Line
-	3555 2630 3850 2630
+	3555 2630 3755 2630
+Wire Wire Line
+	3755 2630 3850 2630
 Connection ~ 3605 2930
 Wire Wire Line
-	3605 4205 3605 2930
-Wire Wire Line
-	3825 4205 3605 4205
-Wire Wire Line
-	3755 3905 3755 2630
-Wire Wire Line
-	3825 3905 3755 3905
+	3605 2930 3605 4445
+Wire Wire Line
+	3605 4445 3825 4445
+Wire Wire Line
+	3755 2630 3755 4145
+Wire Wire Line
+	3755 4145 3825 4145
 Wire Wire Line
 	3555 2430 3850 2430
 Wire Wire Line
-	3825 3505 3825 3705
+	3825 3505 3825 3945
 Wire Wire Line
 	5250 3505 3825 3505
@@
 	5250 3330 5250 3505
 Wire Wire Line
-	5225 3705 5430 3705
-Wire Wire Line
-	5430 3805 5225 3805
-Wire Wire Line
-	5430 3905 5225 3905
+	5225 3945 5430 3945
+Wire Wire Line
+	5430 4045 5225 4045
+Wire Wire Line
+	5430 4145 5225 4145
 Wire Wire Line
 	6865 4150 6865 4555
@@
 	5730 3035 5875 3035
 Wire Wire Line
-	3825 4005 3675 4005
-Wire Wire Line
-	3675 4005 3675 3985
-Wire Wire Line
-	3825 4305 3675 4305
-Wire Wire Line
-	3675 4305 3675 4335
-Wire Wire Line
-	3850 2730 3830 2730
-Wire Wire Line
-	3830 2730 3830 2375
+	3675 4245 3825 4245
+Wire Wire Line
+	3825 4545 3675 4545
+Wire Wire Line
+	3675 4545 3675 5020
+Wire Wire Line
+	3830 2730 3850 2730
+Wire Wire Line
+	3830 2165 3830 2730
 Wire Wire Line
 	3850 3030 3830 3030
 Wire Wire Line
-	3830 3030 3830 3075
+	3830 3030 3830 3155
+Wire Wire Line
+	3830 3155 3830 3255
 Wire Wire Line
 	6545 4150 6545 4230
@@
 Wire Wire Line
 	6945 2395 6340 2395
+$Comp
+L +5V #PWR?
+U 1 1 570CE6BE
+P 4390 2120
+F 0 "#PWR?" H 4390 1970 50  0001 C CNN
+F 1 "+5V" H 4390 2260 50  0000 C CNN
+F 2 "" H 4390 2120 50  0000 C CNN
+F 3 "" H 4390 2120 50  0000 C CNN
+	1    4390 2120
+	1    0    0    -1
+$EndComp
+Wire Wire Line
+	4105 3155 4105 3480
+Wire Wire Line
+	4105 3480 4390 3480
+Wire Wire Line
+	4390 3480 4390 3470
+Wire Wire Line
+	3675 3715 3675 4245
+Wire Wire Line
+	4390 2120 4390 2165
+Wire Wire Line
+	4390 2165 4390 2230
+Wire Wire Line
+	3830 2165 4390 2165
+Connection ~ 4390 2165
+Wire Wire Line
+	4105 3155 3830 3155
+Connection ~ 3830 3155
+Wire Wire Line
+	4365 3685 4365 3715
+Wire Wire Line
+	4365 3715 4365 3745
+$Comp
+L +5V #PWR?
+U 1 1 570D4D3C
+P 4365 3685
+F 0 "#PWR?" H 4365 3535 50  0001 C CNN
+F 1 "+5V" H 4365 3825 50  0000 C CNN
+F 2 "" H 4365 3685 50  0000 C CNN
+F 3 "" H 4365 3685 50  0000 C CNN
+	1    4365 3685
+	1    0    0    -1
+$EndComp
+Wire Wire Line
+	3675 3715 4365 3715
+Connection ~ 4365 3715
+Wire Wire Line
+	4365 4985 4365 5020
+Wire Wire Line
+	4365 5020 4365 5055
+Wire Wire Line
+	3675 5020 4365 5020
+Connection ~ 4365 5020
 $EndSCHEMATC

Commit message: Added files via upload
Changed lines of the file:
@@
 LIBS:valves
 LIBS:WIFIRE
+LIBS:spiflash_16m
 LIBS:НИРС-cache
 EELAYER 25 0
@@
 RCLK
 Wire Wire Line
-	3555 2930 3605 2930
-Wire Wire Line
-	3605 2930 3850 2930
+	3555 2930 3850 2930
 Connection ~ 3755 2630
 Wire Wire Line
-	3555 2630 3755 2630
-Wire Wire Line
-	3755 2630 3850 2630
+	3555 2630 3850 2630
 Connection ~ 3605 2930
 Wire Wire Line
@@
 	3850 3030 3830 3030
 Wire Wire Line
-	3830 3030 3830 3155
-Wire Wire Line
-	3830 3155 3830 3255
+	3830 3030 3830 3255
 Wire Wire Line
 	6545 4150 6545 4230
@@
 	3675 3715 3675 4245
 Wire Wire Line
-	4390 2120 4390 2165
-Wire Wire Line
-	4390 2165 4390 2230
+	4390 2120 4390 2230
 Wire Wire Line
 	3830 2165 4390 2165
@@
 Connection ~ 3830 3155
 Wire Wire Line
-	4365 3685 4365 3715
-Wire Wire Line
-	4365 3715 4365 3745
+	4365 3685 4365 3745
 $Comp
 L +5V #PWR?
@@
 Connection ~ 4365 3715
 Wire Wire Line
-	4365 4985 4365 5020
-Wire Wire Line
-	4365 5020 4365 5055
+	4365 4985 4365 5055
 Wire Wire Line
 	3675 5020 4365 5020

Commit message: Add files via upload
Parts:
- R201, R202, R203, R204, R205, R206, R207, R208: footprint Resistors_SMD:R_0402 -> Resistors_SMD:R_0805
Changed lines of the file:
@@
 LIBS:valves
 LIBS:WIFIRE
-LIBS:spiflash_16m
 LIBS:НИРС-cache
 EELAYER 25 0
@@
 F 0 "R201" V 5540 2265 50  0000 C CNN
 F 1 "68" V 5460 2265 50  0000 C CNN
-F 2 "Resistors_SMD:R_0402" V 5390 2265 50  0001 C CNN
+F 2 "Resistors_SMD:R_0805" V 5390 2265 50  0001 C CNN
 F 3 "" H 5460 2265 50  0000 C CNN
 	1    5460 2265
@@
 F 0 "R207" V 5540 3195 50  0000 C CNN
 F 1 "68" V 5460 3195 50  0000 C CNN
-F 2 "Resistors_SMD:R_0402" V 5390 3195 50  0001 C CNN
+F 2 "Resistors_SMD:R_0805" V 5390 3195 50  0001 C CNN
 F 3 "" H 5460 3195 50  0000 C CNN
 	1    5460 3195
@@
 F 0 "R205" V 5540 2885 50  0000 C CNN
 F 1 "68" V 5460 2885 50  0000 C CNN
-F 2 "Resistors_SMD:R_0402" V 5390 2885 50  0001 C CNN
+F 2 "Resistors_SMD:R_0805" V 5390 2885 50  0001 C CNN
 F 3 "" H 5460 2885 50  0000 C CNN
 	1    5460 2885
@@
 F 0 "R203" V 5540 2575 50  0000 C CNN
 F 1 "68" V 5460 2575 50  0000 C CNN
-F 2 "Resistors_SMD:R_0402" V 5390 2575 50  0001 C CNN
+F 2 "Resistors_SMD:R_0805" V 5390 2575 50  0001 C CNN
 F 3 "" H 5460 2575 50  0000 C CNN
 	1    5460 2575
@@
 F 0 "R202" V 5540 2420 50  0000 C CNN
 F 1 "68" V 5460 2420 50  0000 C CNN
-F 2 "Resistors_SMD:R_0402" V 5390 2420 50  0001 C CNN
+F 2 "Resistors_SMD:R_0805" V 5390 2420 50  0001 C CNN
 F 3 "" H 5460 2420 50  0000 C CNN
 	1    5460 2420
@@
 F 0 "R208" V 5540 3350 50  0000 C CNN
 F 1 "68" V 5460 3350 50  0000 C CNN
-F 2 "Resistors_SMD:R_0402" V 5390 3350 50  0001 C CNN
+F 2 "Resistors_SMD:R_0805" V 5390 3350 50  0001 C CNN
 F 3 "" H 5460 3350 50  0000 C CNN
 	1    5460 3350
@@
 F 0 "R206" V 5540 3040 50  0000 C CNN
 F 1 "68" V 5460 3040 50  0000 C CNN
-F 2 "Resistors_SMD:R_0402" V 5390 3040 50  0001 C CNN
+F 2 "Resistors_SMD:R_0805" V 5390 3040 50  0001 C CNN
 F 3 "" H 5460 3040 50  0000 C CNN
 	1    5460 3040
@@
 F 0 "R204" V 5540 2730 50  0000 C CNN
 F 1 "68" V 5460 2730 50  0000 C CNN
-F 2 "Resistors_SMD:R_0402" V 5390 2730 50  0001 C CNN
+F 2 "Resistors_SMD:R_0805" V 5390 2730 50  0001 C CNN
 F 3 "" H 5460 2730 50  0000 C CNN
 	1    5460 2730
@@
 $EndComp
 $Comp
-L GND #PWR022
+L GND #PWR029
 U 1 1 56F5E482
 P 4365 5055
-F 0 "#PWR022" H 4365 4805 50  0001 C CNN
+F 0 "#PWR029" H 4365 4805 50  0001 C CNN
 F 1 "GND" H 4365 4905 50  0000 C CNN
 F 2 "" H 4365 5055 50  0000 C CNN
@@
 $EndComp
 $Comp
-L GND #PWR023
+L GND #PWR030
 U 1 1 56F5E488
 P 3830 3255
-F 0 "#PWR023" H 3830 3005 50  0001 C CNN
+F 0 "#PWR030" H 3830 3005 50  0001 C CNN
 F 1 "GND" H 3830 3105 50  0000 C CNN
 F 2 "" H 3830 3255 50  0000 C CNN
@@
 	6945 2395 6340 2395
 $Comp
-L +5V #PWR?
+L +5V #PWR031
 U 1 1 570CE6BE
 P 4390 2120
-F 0 "#PWR?" H 4390 1970 50  0001 C CNN
+F 0 "#PWR031" H 4390 1970 50  0001 C CNN
 F 1 "+5V" H 4390 2260 50  0000 C CNN
 F 2 "" H 4390 2120 50  0000 C CNN
@@
 	4365 3685 4365 3745
 $Comp
-L +5V #PWR?
+L +5V #PWR032
 U 1 1 570D4D3C
 P 4365 3685
-F 0 "#PWR?" H 4365 3535 50  0001 C CNN
+F 0 "#PWR032" H 4365 3535 50  0001 C CNN
 F 1 "+5V" H 4365 3825 50  0000 C CNN
 F 2 "" H 4365 3685 50  0000 C CNN
