File: project/file5702498E.sch (KiCad schematic (older format))
At the start: 41 parts

Commit message: Added files via upload
Parts:
- removed Q? (x8): PN2222A, symbol PN2222A
- added Q301, Q302, Q303, Q304, Q305, Q306, Q307, Q308: Tran_8050, TO_SOT_Packages_SMD:SOT-23, symbol Tran_8050
- LED301: renamed from LED?; footprint (none) -> WIFIRE:GNM-7881
- R301, R302, R303, R304, R305, R306, R307, R308, R309, R310, R311, R312, R313, R314, R315, R316, R317, R318, R319, R320, R321, R322, R323, R324, R325, R326, R327, R328, R329, R330, R331, R332: renamed from R?; footprint (none) -> Resistors_SMD:R_0402

Commit message: Add files via upload
Parts:
- R301, R302, R303, R304, R305, R306, R307, R308, R309, R310, R311, R312, R313, R314, R315, R316, R317, R318, R319, R320, R321, R322, R323, R324, R325, R326, R327, R328, R329, R330, R331, R332: footprint Resistors_SMD:R_0402 -> Resistors_SMD:R_0805
